File: nowyprojekt.kicad_pcb (KiCad board)
At the start: 4 copper layers, 75.6 x 70.8 mm, 46 parts, among them J1 Zasilanie, J2 01x03, J3 Conn_01x15_Pin, J4 Conn_01x15_Pin, Q1 BC856, Q2 BC856, Q3 BC856, Q4 BC856, U1 CA56-12SURKWA, U2 ATMEGA328P-AU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

Commit message: latest 04.04.2026r update - text - opis PCB
Parts:
- removed the REF** at (160.1, 84.6)
- moved REF** 6.30 mm to (229.1, 49.6)
- moved REF** 2.90 mm to (160.2, 49.6)
Other:
- board text added: "+"
- board text added: "+5V"
- board text added: "ADC1"
- board text added: "ADC2"
- board text added: "AMS1117 5.0V"
- board text added: "ATmega328p project"
- board text added: "GND"
- board text added: "K"
- board text added: "PB0"
- board text added: "PB1"
- board text added: "PB2"
- board text added: "PB3"
- board text added: "PB4"
- board text added: "PB5"
- board text added: "PC0"
- board text added: "PC1"
- board text added: "PC2"
- board text added: "PC3"
- board text added: "PC4"
- board text added: "PC5"
- board text added: "PC6"
- board text added: "PD0"
- board text added: "PD1"
- board text added: "PD2"
- board text added: "PD3"
- board text added: "PD4"
- board text added: "PD5"
- board text added: "PD6"
- board text added: "PD7"
- board text added: "VIN"
- board text added: "Version 1.00"
- board text added: "made by Adrian L"
- board text added: "max 15V"
- board text removed: "Gnd"
- board text removed: "Vin"
